File: power.kicad_sch (KiCad schematic)
At the start: 23 parts, among them U1 LM27313XMF, U2 LP2985-3.3

Commit message: C3,5,7,17 had LCSC changed to rev 1.1
Parts:
- C3: footprint Capacitor_SMD:C_0402_1005Metric_Pad0.74x0.62mm_HandSolder -> Capacitor_SMD:C_0805_2012Metric_Pad1.18x1.45mm_HandSolder
- C5: LCSC C1779 -> C106859
Changed lines of the file:
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@@
 			)
 		)
-		(property "LCSC" "C1779"
+		(property "LCSC" "C106859"
 			(at 91.44 124.46 90)
 			(effects
@@
 			)
 		)
-		(property "Footprint" "Capacitor_SMD:C_0402_1005Metric_Pad0.74x0.62mm_HandSolder"
+		(property "Footprint" "Capacitor_SMD:C_0805_2012Metric_Pad1.18x1.45mm_HandSolder"
 			(at 109.982 74.93 90)
 			(effects

Commit message: Wrong LCSC part number for 3.3V regulator. BOOT1 needs to be held LOW not HIGH.
Parts:
- U2: LCSC C109382 -> C129375
Changed lines of the file:
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@@
 			)
 		)
-		(property "LCSC" "C109382"
+		(property "LCSC" "C129375"
 			(at 64.77 119.38 0)
 			(effects
