File: uController.kicad_sch (KiCad schematic)
At the start: 35 parts, among them J1 USB_B_Micro, J2 TagConnectTC2050, SW1 SW_Push, SW2 SW_Push, U3 STM32F411RETx, U4 93LC66AT-IOT, Y1 16M 20pF 3225

Commit message: C3,5,7,17 had LCSC changed to rev 1.1
Parts:
- C17, C7: LCSC C1779 -> C106859
Changed lines of the file:
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@@
 			)
 		)
-		(property "LCSC" "C1779"
+		(property "LCSC" "C106859"
 			(at 119.38 129.54 90)
 			(effects
@@
 			)
 		)
-		(property "LCSC" "C1779"
+		(property "LCSC" "C106859"
 			(at 120.65 27.94 90)
 			(effects

Commit message: Wrong LCSC part number for 3.3V regulator. BOOT1 needs to be held LOW not HIGH.
Parts:
- added R17: 100, Resistor_SMD:R_0402_1005Metric_Pad0.72x0.64mm_HandSolder, symbol Device:R
- R12: now not fitted
Connections:
- net BOOT1: now also R17.1
- net GND: now also R17.2
Other:
- note added: "ERRATA: BOOT1 should be held LOW for DFU to work. PCB has NOT been updated!"
Changed lines of the file:
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@@
 	)
 	(junction
+		(at 189.23 105.41)
+		(diameter 0)
+		(color 0 0 0 0)
+	)
+	(junction
 		(at 144.78 50.8)
 		(diameter 0)
@@
 	(wire
 		(pts
+			(xy 189.23 105.41) (xy 195.58 105.41)
+		)
+		(stroke
+			(width 0)
+			(type default)
+		)
+	)
+	(wire
+		(pts
 			(xy 185.42 80.01) (xy 190.5 80.01)
 		)
@@
 	(wire
 		(pts
+			(xy 205.74 105.41) (xy 203.2 105.41)
+		)
+		(stroke
+			(width 0)
+			(type default)
+		)
+	)
+	(wire
+		(pts
 			(xy 153.67 38.1) (xy 153.67 49.53)
 		)
@@
 	(wire
 		(pts
+			(xy 205.74 106.68) (xy 205.74 105.41)
+		)
+		(stroke
+			(width 0)
+			(type default)
+		)
+	)
+	(wire
+		(pts
 			(xy 100.33 62.23) (xy 101.6 62.23)
 		)
@@
 		)
 	)
+	(rectangle
+		(start 208.28 95.25)
+		(end 257.81 110.49)
+		(stroke
+			(width 0)
+			(type default)
+		)
+		(fill
+			(type color)
+			(color 160 160 160 1)
+		)
+	)
 	(text "RESET"
 		(exclude_from_sim no)
@@
 		)
 	)
+	(text "ERRATA:\nBOOT1 should be held LOW for DFU to work.\nPCB has NOT been updated!"
+		(exclude_from_sim no)
+		(at 231.902 102.616 0)
+		(effects
+			(font
+				(size 1.27 1.27)
+				(thickness 0.254)
+				(bold yes)
+				(color 0 0 0 1)
+			)
+		)
+	)
 	(label "SPI2_MOSI"
 		(at 58.42 149.86 0)
@@
 	(symbol
 		(lib_id "power:GND")
+		(at 205.74 106.68 0)
+		(unit 1)
+		(exclude_from_sim no)
+		(in_bom yes)
+		(on_board yes)
+		(dnp no)
+		(property "Reference" "#PWR049"
+			(at 205.74 113.03 0)
+			(effects
+				(font
+					(size 1.27 1.27)
+				)
+				(hide yes)
+			)
+		)
+		(property "Value" "GND"
+			(at 203.708 109.728 0)
+			(effects
+				(font
+					(size 1.27 1.27)
+				)
+				(hide yes)
+			)
+		)
+		(property "Footprint" ""
+			(at 205.74 106.68 0)
+			(effects
+				(font
+					(size 1.27 1.27)
+				)
+				(hide yes)
+			)
+		)
+		(property "Datasheet" ""
+			(at 205.74 106.68 0)
+			(effects
+				(font
+					(size 1.27 1.27)
+				)
+				(hide yes)
+			)
+		)
+		(property "Description" "Power symbol creates a global label with name \"GND\" , ground"
+			(at 205.74 106.68 0)
+			(effects
+				(font
+					(size 1.27 1.27)
+				)
+				(hide yes)
+			)
+		)
+		(pin "1"
+		)
+		(instances
+			(project "USB_8769M"
+				(path "/05725277-f916-41de-9b08-3e24bb187c9c/a7dd05cd-dc8b-4c10-b82d-5446c7ae4287"
+					(reference "#PWR049")
+					(unit 1)
+				)
+			)
+		)
+	)
+	(symbol
+		(lib_id "power:GND")
 		(at 48.26 44.45 0)
 		(unit 1)
@@
 	)
 	(symbol
+		(lib_id "Device:R")
+		(at 199.39 105.41 90)
+		(unit 1)
+		(exclude_from_sim no)
+		(in_bom yes)
+		(on_board yes)
+		(dnp no)
+		(fields_autoplaced yes)
+		(property "Reference" "R17"
+			(at 199.39 99.06 90)
+			(effects
+				(font
+					(size 1.27 1.27)
+				)
+			)
+		)
+		(property "Value" "100"
+			(at 199.39 101.6 90)
+			(effects
+				(font
+					(size 1.27 1.27)
+				)
+			)
+		)
+		(property "Footprint" "Resistor_SMD:R_0402_1005Metric_Pad0.72x0.64mm_HandSolder"
+			(at 199.39 107.188 90)
+			(effects
+				(font
+					(size 1.27 1.27)
+				)
+				(hide yes)
+			)
+		)
+		(property "Datasheet" "~"
+			(at 199.39 105.41 0)
+			(effects
+				(font
+					(size 1.27 1.27)
+				)
+				(hide yes)
+			)
+		)
+		(property "Description" "Resistor"
+			(at 199.39 105.41 0)
+			(effects
+				(font
+					(size 1.27 1.27)
+				)
+				(hide yes)
+			)
+		)
+		(property "LCSC" "C25076"
+			(at 199.39 105.41 0)
+			(effects
+				(font
+					(size 1.27 1.27)
+				)
+				(hide yes)
+			)
+		)
+		(pin "1"
+		)
+		(pin "2"
+		)
+		(instances
+			(project "USB_8769M"
+				(path "/05725277-f916-41de-9b08-3e24bb187c9c/a7dd05cd-dc8b-4c10-b82d-5446c7ae4287"
+					(reference "R17")
+					(unit 1)
+				)
+			)
+		)
+	)
+	(symbol
 		(lib_id "power:GND")
 		(at 115.57 27.94 0)
@@
 		(in_bom yes)
 		(on_board yes)
-		(dnp no)
+		(dnp yes)
 		(fields_autoplaced yes)
 		(property "Reference" "R12"
